Commit message: fix base name

File: legged_gym/resources/robots/go2/urdf/go2.urdf (robot description, URDF)
Before this commit: robot go2, 42 links, 41 joints
Links:
- removed link trunk
- added link base, mass 6.921; collision box size=0.3762 0.0935 0.114; visual mesh filename=./dae/base.dae
Joints:
- joint FL_hip_joint: parent trunk -> base
- joint FL_hip_rotor_joint: parent trunk -> base
- joint FR_hip_joint: parent trunk -> base
- joint FR_hip_rotor_joint: parent trunk -> base
- joint Head_upper_joint: parent trunk -> base
- joint RL_hip_joint: parent trunk -> base
- joint RL_hip_rotor_joint: parent trunk -> base
- joint RR_hip_joint: parent trunk -> base
- joint RR_hip_rotor_joint: parent trunk -> base
- joint front_camera_joint: parent trunk -> base
- joint imu_joint: parent trunk -> base
- joint radar_joint: parent trunk -> base
